File: hw/candled/power.sch (KiCad schematic (older format))
At the start: 6 parts, among them J4 5V, U2 LM2596

Commit message: add one-pin TX/RX schematic design
Parts:
- L1: value 68μH -> 68μH @ 3A
Changed lines of the file:
@@
 P 7200 3950
 F 0 "L1" V 7300 4000 50  0000 C CNN
-F 1 "68μH" V 7100 3950 50  0000 C CNN
+F 1 "68μH @ 3A" V 7100 3950 50  0000 C CNN
 F 2 "" H 7200 3950 50  0001 C CNN
 F 3 "~" H 7200 3950 50  0001 C CNN
